Commit message: sensor data added

File: body.urdf (robot description, URDF)
Before this commit: robot robot, 1 links, 0 joints
Links:
- added link BackLeg, mass 1; collision box size=1.0 1.0 1.0; visual box size=1.0 1.0 1.0
- added link FrontLeg, mass 1; collision box size=1.0 1.0 1.0; visual box size=1.0 1.0 1.0
Joints:
- added joint Torso_BackLeg: type revolute, parent Torso, child BackLeg, origin xyz=1.0 0.0 1.0 rpy=0 0 0, axis 0 1 0, limit lower=-3.14159 upper=3.14159 effort=0.0 velocity=0.0
- added joint Torso_FrontLeg: type revolute, parent Torso, child FrontLeg, origin xyz=2.0 0.0 1.0 rpy=0 0 0, axis 0 1 0, limit lower=-3.14159 upper=3.14159 effort=0.0 velocity=0.0

Commit message: add limbs

File: body.urdf (robot description, URDF)
Before this commit: robot robot, 3 links, 2 joints
Links:
- link BackLeg: geometry collision box size=0.2 1 0.2; visual box size=0.2 1 0.2
- link FrontLeg: geometry collision box size=0.2 1 0.2; visual box size=0.2 1 0.2
Joints:
- joint Torso_BackLeg: axis 0 1 0 -> 1 0 0; origin xyz=1.0 0.0 1.0 rpy=0 0 0 -> xyz=0.0 -0.5 1.0 rpy=0 0 0
- joint Torso_FrontLeg: axis 0 1 0 -> 1 0 0; origin xyz=2.0 0.0 1.0 rpy=0 0 0 -> xyz=0.0 0.5 1.0 rpy=0 0 0

Commit message: fixed sensors and desired angle

File: body.urdf (robot description, URDF)
Before this commit: robot robot, 3 links, 2 joints
Links:
- added link BackLowerLeg, mass 1; collision box size=0.2 0.2 1.0; visual box size=0.2 0.2 1.0
- added link FrontLowerLeg, mass 1; collision box size=0.2 0.2 1.0; visual box size=0.2 0.2 1.0
- added link LeftLeg, mass 1; collision box size=1.0 0.2 0.2; visual box size=1.0 0.2 0.2
- added link LeftLowerLeg, mass 1; collision box size=0.2 0.2 1.0; visual box size=0.2 0.2 1.0
- added link RightLeg, mass 1; collision box size=1.0 0.2 0.2; visual box size=1.0 0.2 0.2
- added link RightLowerLeg, mass 1; collision box size=0.2 0.2 1.0; visual box size=0.2 0.2 1.0
Joints:
- added joint BackLeg_BackLowerLeg: type revolute, parent BackLeg, child BackLowerLeg, origin xyz=0.0 -1.0 0.0 rpy=0 0 0, axis 1 0 0, limit lower=-3.14159 upper=3.14159 effort=0.0 velocity=0.0
- added joint FrontLeg_FrontLowerLeg: type revolute, parent FrontLeg, child FrontLowerLeg, origin xyz=0.0 1.0 0.0 rpy=0 0 0, axis 1 0 0, limit lower=-3.14159 upper=3.14159 effort=0.0 velocity=0.0
- added joint LeftLeg_LeftLowerLeg: type revolute, parent LeftLeg, child LeftLowerLeg, origin xyz=-1.0 0.0 0.0 rpy=0 0 0, axis 0 1 0, limit lower=-3.14159 upper=3.14159 effort=0.0 velocity=0.0
- added joint RightLeg_RightLowerLeg: type revolute, parent RightLeg, child RightLowerLeg, origin xyz=1.0 0.0 0.0 rpy=0 0 0, axis 0 1 0, limit lower=-3.14159 upper=3.14159 effort=0.0 velocity=0.0
- added joint Torso_LeftLeg: type revolute, parent Torso, child LeftLeg, origin xyz=-0.5 0.0 1.0 rpy=0 0 0, axis 0 1 0, limit lower=-3.14159 upper=3.14159 effort=0.0 velocity=0.0
- added joint Torso_RightLeg: type revolute, parent Torso, child RightLeg, origin xyz=0.5 0.0 1.0 rpy=0 0 0, axis 0 1 0, limit lower=-3.14159 upper=3.14159 effort=0.0 velocity=0.0

Commit message: torso and upper legs

File: body.urdf (robot description, URDF)
Before this commit: robot robot, 9 links, 8 joints
Links:
- removed link BackLowerLeg
- removed link FrontLowerLeg
- removed link LeftLeg
- removed link LeftLowerLeg
- removed link RightLeg
- removed link RightLowerLeg
- link BackLeg: geometry collision box size=0.4 0.4 1.25; visual box size=0.4 0.4 1.25
- link FrontLeg: geometry collision box size=0.4 0.4 1.25; visual box size=0.4 0.4 1.25
- link Torso: geometry collision box size=0.75 1.0 1.0; visual box size=0.75 1.0 1.0
Joints:
- removed joint BackLeg_BackLowerLeg
- removed joint FrontLeg_FrontLowerLeg
- removed joint LeftLeg_LeftLowerLeg
- removed joint RightLeg_RightLowerLeg
- removed joint Torso_LeftLeg
- removed joint Torso_RightLeg
- joint Torso_BackLeg: axis 1 0 0 -> 0 1 0; origin xyz=0.0 -0.5 1.0 rpy=0 0 0 -> xyz=0.0 0.5 1.0 rpy=0 0 0
- joint Torso_FrontLeg: axis 1 0 0 -> 0 1 0

Commit message: biped form and +x optimize

File: body.urdf (robot description, URDF)
Before this commit: robot robot, 3 links, 2 joints
Links:
- removed link BackLeg
- removed link FrontLeg
- added link LeftFoot, mass 1; collision box size=0.6 0.3 0.25; visual box size=0.6 0.3 0.25
- added link LeftLeg, mass 1; collision box size=0.4 0.3 1.25; visual box size=0.4 0.3 1.25
- added link LeftLowerLeg, mass 1; collision box size=0.4 0.3 1.25; visual box size=0.4 0.3 1.25
- added link RightFoot, mass 1; collision box size=0.6 0.3 0.25; visual box size=0.6 0.3 0.25
- added link RightLeg, mass 1; collision box size=0.4 0.3 1.25; visual box size=0.4 0.3 1.25
- added link RightLowerLeg, mass 1; collision box size=0.4 0.3 1.25; visual box size=0.4 0.3 1.25
Joints:
- removed joint Torso_BackLeg
- removed joint Torso_FrontLeg
- added joint LeftLeg_LeftLowerLeg: type revolute, parent LeftLeg, child LeftLowerLeg, origin xyz=0.0 0.0 -0.5 rpy=0 0 0, axis 0 1 0, limit lower=-3.14159 upper=3.14159 effort=0.0 velocity=0.0
- added joint LeftLowerLeg_LeftFoot: type revolute, parent LeftLowerLeg, child LeftFoot, origin xyz=0.0 0.0 -0.6 rpy=0 0 0, axis 0 1 0, limit lower=-3.14159 upper=3.14159 effort=0.0 velocity=0.0
- added joint RightLeg_RightLowerLeg: type revolute, parent RightLeg, child RightLowerLeg, origin xyz=0.0 0.0 -0.5 rpy=0 0 0, axis 0 1 0, limit lower=-3.14159 upper=3.14159 effort=0.0 velocity=0.0
- added joint RightLowerLeg_RightFoot: type revolute, parent RightLowerLeg, child RightFoot, origin xyz=0.0 0.0 -0.6 rpy=0 0 0, axis 0 1 0, limit lower=-3.14159 upper=3.14159 effort=0.0 velocity=0.0
- added joint Torso_LeftLeg: type revolute, parent Torso, child LeftLeg, origin xyz=0.0 0.5 1.75 rpy=0 0 0, axis 0 1 0, limit lower=-3.14159 upper=3.14159 effort=0.0 velocity=0.0
- added joint Torso_RightLeg: type revolute, parent Torso, child RightLeg, origin xyz=0.0 -0.5 1.75 rpy=0 0 0, axis 0 1 0, limit lower=-3.14159 upper=3.14159 effort=0.0 velocity=0.0

Commit message: adjust proportions

File: body.urdf (robot description, URDF)
Before this commit: robot robot, 7 links, 6 joints
Links:
- link LeftFoot: geometry collision box size=0.85 0.45 0.15; visual box size=0.85 0.45 0.15
- link LeftLeg: geometry collision box size=0.4 0.3 1.75; visual box size=0.4 0.3 1.75
- link RightFoot: geometry collision box size=0.85 0.45 0.15; visual box size=0.85 0.45 0.15
- link RightLeg: geometry collision box size=0.4 0.3 1.75; visual box size=0.4 0.3 1.75
- link Torso: geometry collision box size=0.65 0.85 0.75; visual box size=0.65 0.85 0.75
Joints:
- joint LeftLeg_LeftLowerLeg: origin xyz=0.0 0.0 -0.5 rpy=0 0 0 -> xyz=0.0 0.0 -0.79 rpy=0 0 0
- joint LeftLowerLeg_LeftFoot: origin xyz=0.0 0.0 -0.6 rpy=0 0 0 -> xyz=0.1 0.0 -0.6 rpy=0 0 0
- joint RightLeg_RightLowerLeg: origin xyz=0.0 0.0 -0.5 rpy=0 0 0 -> xyz=0.0 0.0 -0.79 rpy=0 0 0
- joint RightLowerLeg_RightFoot: origin xyz=0.0 0.0 -0.6 rpy=0 0 0 -> xyz=0.1 0.0 -0.6 rpy=0 0 0
- joint Torso_LeftLeg: origin xyz=0.0 0.5 1.75 rpy=0 0 0 -> xyz=0.0 0.3 2.2 rpy=0 0 0
- joint Torso_RightLeg: origin xyz=0.0 -0.5 1.75 rpy=0 0 0 -> xyz=0.0 -0.3 2.2 rpy=0 0 0

Commit message: tryna fix the body...

File: body.urdf (robot description, URDF)
Before this commit: robot robot, 7 links, 6 joints
Links:
- link LeftLowerLeg: geometry collision box size=0.4 0.3 1.3; visual box size=0.4 0.3 1.3
- link RightLowerLeg: geometry collision box size=0.4 0.3 1.3; visual box size=0.4 0.3 1.3
- link Torso: geometry collision box size=0.55 0.85 0.55; visual box size=0.55 0.85 0.55

Commit message: stuggling...

File: body.urdf (robot description, URDF)
Before this commit: robot robot, 7 links, 6 joints
Joints:
- joint LeftLeg_LeftLowerLeg: limit lower=-3.14159 upper=3.14159 effort=0.0 velocity=0.0 -> lower=-0.5235833333333334 upper=0.0 effort=0.0 velocity=0.0
- joint LeftLowerLeg_LeftFoot: limit lower=-3.14159 upper=3.14159 effort=0.0 velocity=0.0 -> lower=-0.5235833333333334 upper=0.5235833333333334 effort=0.0 velocity=0.0; origin xyz=0.1 0.0 -0.6 rpy=0 0 0 -> xyz=0.0 0.0 -0.6 rpy=0 0 0
- joint RightLeg_RightLowerLeg: limit lower=-3.14159 upper=3.14159 effort=0.0 velocity=0.0 -> lower=-0.5235833333333334 upper=0.0 effort=0.0 velocity=0.0
- joint RightLowerLeg_RightFoot: limit lower=-3.14159 upper=3.14159 effort=0.0 velocity=0.0 -> lower=-0.5235833333333334 upper=0.5235833333333334 effort=0.0 velocity=0.0; origin xyz=0.1 0.0 -0.6 rpy=0 0 0 -> xyz=0.0 0.0 -0.6 rpy=0 0 0
- joint Torso_LeftLeg: limit lower=-3.14159 upper=3.14159 effort=0.0 velocity=0.0 -> lower=-0.5235833333333334 upper=0.5235833333333334 effort=0.0 velocity=0.0; origin xyz=0.0 0.3 2.2 rpy=0 0 0 -> xyz=0.0 0.3 3.25 rpy=0 0 0
- joint Torso_RightLeg: limit lower=-3.14159 upper=3.14159 effort=0.0 velocity=0.0 -> lower=-0.5235833333333334 upper=0.5235833333333334 effort=0.0 velocity=0.0; origin xyz=0.0 -0.3 2.2 rpy=0 0 0 -> xyz=0.0 -0.3 3.25 rpy=0 0 0

Commit message: Changed body

File: body.urdf (robot description, URDF)
Before this commit: robot robot, 7 links, 6 joints
Links:
- link LeftFoot: geometry collision box size=0.575 0.575 0.125; visual box size=0.575 0.575 0.125
- link LeftLeg: geometry collision box size=0.35 0.35 2.25; visual box size=0.35 0.35 2.25
- link LeftLowerLeg: geometry collision box size=0.35 0.35 1.625; visual box size=0.35 0.35 1.625
- link RightFoot: geometry collision box size=0.575 0.575 0.125; visual box size=0.575 0.575 0.125
- link RightLeg: geometry collision box size=0.35 0.35 2.25; visual box size=0.35 0.35 2.25
- link RightLowerLeg: geometry collision box size=0.35 0.35 1.625; visual box size=0.35 0.35 1.625
- link Torso: geometry collision box size=0.375 0.875 0.375; visual box size=0.375 0.875 0.375
Joints:
- joint LeftLeg_LeftLowerLeg: limit lower=-0.5235833333333334 upper=0.0 effort=0.0 velocity=0.0 -> lower=0.0 upper=3.1415 effort=0.0 velocity=0.0; origin xyz=0.0 0.0 -0.79 rpy=0 0 0 -> xyz=0.0 0.0 -2.25 rpy=0 0 0
- joint LeftLowerLeg_LeftFoot: limit lower=-0.5235833333333334 upper=0.5235833333333334 effort=0.0 velocity=0.0 -> lower=-0.785375 upper=0.785375 effort=0.0 velocity=0.0; origin xyz=0.0 0.0 -0.6 rpy=0 0 0 -> xyz=0.0 0.0 -1.625 rpy=0 0 0
- joint RightLeg_RightLowerLeg: limit lower=-0.5235833333333334 upper=0.0 effort=0.0 velocity=0.0 -> lower=0.0 upper=3.1415 effort=0.0 velocity=0.0; origin xyz=0.0 0.0 -0.79 rpy=0 0 0 -> xyz=0.0 0.0 -2.25 rpy=0 0 0
- joint RightLowerLeg_RightFoot: limit lower=-0.5235833333333334 upper=0.5235833333333334 effort=0.0 velocity=0.0 -> lower=-0.785375 upper=0.785375 effort=0.0 velocity=0.0; origin xyz=0.0 0.0 -0.6 rpy=0 0 0 -> xyz=0.0 0.0 -1.625 rpy=0 0 0
- joint Torso_LeftLeg: limit lower=-0.5235833333333334 upper=0.5235833333333334 effort=0.0 velocity=0.0 -> lower=-0.785375 upper=0.785375 effort=0.0 velocity=0.0; origin xyz=0.0 0.3 3.25 rpy=0 0 0 -> xyz=0.0 0.375 4.0 rpy=0 0 0
- joint Torso_RightLeg: limit lower=-0.5235833333333334 upper=0.5235833333333334 effort=0.0 velocity=0.0 -> lower=-0.785375 upper=0.785375 effort=0.0 velocity=0.0; origin xyz=0.0 -0.3 3.25 rpy=0 0 0 -> xyz=0.0 -0.375 4.0 rpy=0 0 0

Commit message: struggling w angles...

File: body.urdf (robot description, URDF)
Before this commit: robot robot, 7 links, 6 joints
Links:
- link LeftFoot: geometry collision box size=0.475 0.475 0.125; visual box size=0.475 0.475 0.125
- link LeftLeg: geometry collision box size=0.25 0.25 2.25; visual box size=0.25 0.25 2.25
- link LeftLowerLeg: geometry collision box size=0.25 0.25 1.625; visual box size=0.25 0.25 1.625
- link RightFoot: geometry collision box size=0.475 0.475 0.125; visual box size=0.475 0.475 0.125
- link RightLeg: geometry collision box size=0.25 0.25 2.25; visual box size=0.25 0.25 2.25
- link RightLowerLeg: geometry collision box size=0.25 0.25 1.625; visual box size=0.25 0.25 1.625
- link Torso: geometry collision box size=0.8 1.0 0.5; visual box size=0.8 1.0 0.5
Joints:
- joint LeftLeg_LeftLowerLeg: limit lower=0.0 upper=3.1415 effort=0.0 velocity=0.0 -> lower=0.0 upper=0.785375 effort=0.0 velocity=0.0
- joint LeftLowerLeg_LeftFoot: limit lower=-0.785375 upper=0.785375 effort=0.0 velocity=0.0 -> lower=-0.785375 upper=1.57075 effort=0.0 velocity=0.0
- joint RightLeg_RightLowerLeg: limit lower=0.0 upper=3.1415 effort=0.0 velocity=0.0 -> lower=0.0 upper=0.785375 effort=0.0 velocity=0.0
- joint RightLowerLeg_RightFoot: limit lower=-0.785375 upper=0.785375 effort=0.0 velocity=0.0 -> lower=-0.785375 upper=1.57075 effort=0.0 velocity=0.0
- joint Torso_LeftLeg: limit lower=-0.785375 upper=0.785375 effort=0.0 velocity=0.0 -> lower=0.3926875 upper=-0.3926875 effort=0.0 velocity=0.0; origin xyz=0.0 0.375 4.0 rpy=0 0 0 -> xyz=0.0 0.5 4.0 rpy=0 0 0
- joint Torso_RightLeg: limit lower=-0.785375 upper=0.785375 effort=0.0 velocity=0.0 -> lower=-0.3926875 upper=0.3926875 effort=0.0 velocity=0.0; origin xyz=0.0 -0.375 4.0 rpy=0 0 0 -> xyz=0.0 -0.5 4.0 rpy=0 0 0

Commit message: add upper body

File: body.urdf (robot description, URDF)
Before this commit: robot robot, 7 links, 6 joints
Links:
- removed link Torso
- added link Hips, mass 1; collision box size=0.8 1.0 0.5; visual box size=0.8 1.0 0.5
- added link LeftLowerArm, mass 1; collision box size=0.35 0.35 0.75; visual box size=0.35 0.35 0.75
- added link LeftShoulder, mass 1; collision box size=0.65 1.125 0.25; visual box size=0.65 1.125 0.25
- added link LeftUpperArm, mass 1; collision box size=0.45 0.45 1.0; visual box size=0.45 0.45 1.0
- added link LowerTorso, mass 1; collision box size=0.675 0.875 0.25; visual box size=0.675 0.875 0.25
- added link MidTorso, mass 1; collision box size=0.55 0.75 0.25; visual box size=0.55 0.75 0.25
- added link RightLowerArm, mass 1; collision box size=0.35 0.35 0.75; visual box size=0.35 0.35 0.75
- added link RightShoulder, mass 1; collision box size=0.65 1.125 0.25; visual box size=0.65 1.125 0.25
- added link RightUpperArm, mass 1; collision box size=0.45 0.45 1.0; visual box size=0.45 0.45 1.0
- added link UpperTorso, mass 1; collision box size=0.65 0.85 0.5; visual box size=0.65 0.85 0.5
- link LeftFoot: geometry collision box size=0.675 0.675 0.225; visual box size=0.675 0.675 0.225
- link LeftLeg: geometry collision box size=0.45 0.45 2.25; visual box size=0.45 0.45 2.25
- link LeftLowerLeg: geometry collision box size=0.35 0.35 1.625; visual box size=0.35 0.35 1.625
- link RightFoot: geometry collision box size=0.675 0.675 0.225; visual box size=0.675 0.675 0.225
- link RightLeg: geometry collision box size=0.45 0.45 2.25; visual box size=0.45 0.45 2.25
- link RightLowerLeg: geometry collision box size=0.35 0.35 1.625; visual box size=0.35 0.35 1.625
Joints:
- removed joint Torso_LeftLeg
- removed joint Torso_RightLeg
- added joint Hips_LeftLeg: type revolute, parent Hips, child LeftLeg, origin xyz=0.0 0.5 4.0 rpy=0 0 0, axis 0 1 0, limit lower=-0.31415000000000004 upper=0.31415000000000004 effort=0.0 velocity=0.0
- added joint Hips_LowerTorso: type revolute, parent Hips, child LowerTorso, origin xyz=0.0 0.0 4.25 rpy=0 0 0, axis 0 1 0, limit lower=-0.2617916666666667 upper=0.2617916666666667 effort=0.0 velocity=0.0
- added joint Hips_RightLeg: type revolute, parent Hips, child RightLeg, origin xyz=0.0 -0.5 4.0 rpy=0 0 0, axis 0 1 0, limit lower=-0.31415000000000004 upper=0.31415000000000004 effort=0.0 velocity=0.0
- added joint LeftShoulder_LeftUpperArm: type revolute, parent LeftShoulder, child LeftUpperArm, origin xyz=0.0 -1.125 0.0 rpy=0 0 0, axis 1 1 0, limit lower=-0.31415000000000004 upper=0.31415000000000004 effort=0.0 velocity=0.0
- added joint LeftUpperArm_LeftLowerArm: type revolute, parent LeftUpperArm, child LeftLowerArm, origin xyz=0.0 0.0 -0.875 rpy=0 0 0, axis 0 1 0, limit lower=-0.31415000000000004 upper=0.0 effort=0.0 velocity=0.0
- added joint LowerTorso_MidTorso: type revolute, parent LowerTorso, child MidTorso, origin xyz=0.0 0.0 0.25 rpy=0 0 0, axis 0 1 0, limit lower=0.0 upper=0.0 effort=0.0 velocity=0.0
- added joint MidTorso_UpperTorso: type revolute, parent MidTorso, child UpperTorso, origin xyz=0.0 0.0 0.25 rpy=0 0 0, axis 0 1 0, limit lower=-0.2617916666666667 upper=0.2617916666666667 effort=0.0 velocity=0.0
- added joint RightShoulder_RightUpperArm: type revolute, parent RightShoulder, child RightUpperArm, origin xyz=0.0 1.125 0.0 rpy=0 0 0, axis 1 1 0, limit lower=-0.31415000000000004 upper=0.31415000000000004 effort=0.0 velocity=0.0
- added joint RightUpperArm_RightLowerArm: type revolute, parent RightUpperArm, child RightLowerArm, origin xyz=0.0 0.0 -0.875 rpy=0 0 0, axis 0 1 0, limit lower=-0.31415000000000004 upper=0.0 effort=0.0 velocity=0.0
- added joint UpperTorso_LeftShoulder: type revolute, parent UpperTorso, child LeftShoulder, origin xyz=0.0 0.0 0.625 rpy=0 0 0, axis 0 0 1, limit lower=0.0 upper=0.0 effort=0.0 velocity=0.0
- added joint UpperTorso_RightShoulder: type revolute, parent UpperTorso, child RightShoulder, origin xyz=0.0 0.0 0.625 rpy=0 0 0, axis 0 0 1, limit lower=0.0 upper=0.0 effort=0.0 velocity=0.0

Commit message: mass

File: body.urdf (robot description, URDF)
Before this commit: robot robot, 16 links, 15 joints
Links:
- link Hips: mass 1 -> 2.5
- link LeftFoot: mass 1 -> 1.25
- link LeftLeg: mass 1 -> 3
- link LeftLowerLeg: mass 1 -> 1.5
- link LeftUpperArm: mass 1 -> 1.5
- link RightFoot: mass 1 -> 1.25
- link RightLeg: mass 1 -> 3
- link RightLowerLeg: mass 1 -> 1.5
- link RightUpperArm: mass 1 -> 1.5
Joints:
- joint Hips_LeftLeg: limit lower=-0.31415000000000004 upper=0.31415000000000004 effort=0.0 velocity=0.0 -> lower=-0.785375 upper=0.785375 effort=0.0 velocity=0.0
- joint Hips_RightLeg: limit lower=-0.31415000000000004 upper=0.31415000000000004 effort=0.0 velocity=0.0 -> lower=-0.785375 upper=0.785375 effort=0.0 velocity=0.0
- joint LeftLeg_LeftLowerLeg: limit lower=0.0 upper=0.785375 effort=0.0 velocity=0.0 -> lower=0.0 upper=1.57075 effort=0.0 velocity=0.0
- joint LeftLowerLeg_LeftFoot: limit lower=-0.785375 upper=1.57075 effort=0.0 velocity=0.0 -> lower=-0.31415000000000004 upper=0.0 effort=0.0 velocity=0.0
- joint LeftShoulder_LeftUpperArm: limit lower=-0.31415000000000004 upper=0.31415000000000004 effort=0.0 velocity=0.0 -> lower=0.3926875 upper=-0.3926875 effort=0.0 velocity=0.0
- joint RightLeg_RightLowerLeg: limit lower=0.0 upper=0.785375 effort=0.0 velocity=0.0 -> lower=0.0 upper=1.57075 effort=0.0 velocity=0.0
- joint RightLowerLeg_RightFoot: limit lower=-0.785375 upper=1.57075 effort=0.0 velocity=0.0 -> lower=-0.31415000000000004 upper=0.0 effort=0.0 velocity=0.0
- joint RightShoulder_RightUpperArm: limit lower=-0.31415000000000004 upper=0.31415000000000004 effort=0.0 velocity=0.0 -> lower=-0.3926875 upper=0.3926875 effort=0.0 velocity=0.0

Commit message: save values robot

File: body.urdf (robot description, URDF)
Before this commit: robot robot, 16 links, 15 joints
Links:
- link LowerTorso: mass 1 -> 1.25

Commit message: visualizer

File: body.urdf (robot description, URDF)
Before this commit: robot robot, 16 links, 15 joints
Links:
- link LeftFoot: mass 1.25 -> 1
- link LeftLeg: mass 3 -> 2.75
- link LeftLowerArm: mass 1 -> 1.5
- link RightFoot: mass 1.25 -> 1
- link RightLeg: mass 3 -> 2.75
- link RightLowerArm: mass 1 -> 1.5
Joints:
- joint Hips_LeftLeg: limit lower=-0.785375 upper=0.785375 effort=0.0 velocity=0.0 -> lower=-1.57075 upper=1.57075 effort=0.0 velocity=0.0
- joint Hips_RightLeg: limit lower=-0.785375 upper=0.785375 effort=0.0 velocity=0.0 -> lower=-1.57075 upper=1.57075 effort=0.0 velocity=0.0
- joint LeftLeg_LeftLowerLeg: limit lower=0.0 upper=1.57075 effort=0.0 velocity=0.0 -> lower=0.0 upper=3.1415 effort=0.0 velocity=0.0
- joint LeftLowerLeg_LeftFoot: limit lower=-0.31415000000000004 upper=0.0 effort=0.0 velocity=0.0 -> lower=-0.785375 upper=0.3926875 effort=0.0 velocity=0.0
- joint LeftShoulder_LeftUpperArm: limit lower=0.3926875 upper=-0.3926875 effort=0.0 velocity=0.0 -> lower=0.785375 upper=-0.785375 effort=0.0 velocity=0.0
- joint LeftUpperArm_LeftLowerArm: limit lower=-0.31415000000000004 upper=0.0 effort=0.0 velocity=0.0 -> lower=-0.5235833333333334 upper=0.0 effort=0.0 velocity=0.0
- joint RightLeg_RightLowerLeg: limit lower=0.0 upper=1.57075 effort=0.0 velocity=0.0 -> lower=0.0 upper=3.1415 effort=0.0 velocity=0.0
- joint RightLowerLeg_RightFoot: limit lower=-0.31415000000000004 upper=0.0 effort=0.0 velocity=0.0 -> lower=-0.785375 upper=0.3926875 effort=0.0 velocity=0.0
- joint RightShoulder_RightUpperArm: limit lower=-0.3926875 upper=0.3926875 effort=0.0 velocity=0.0 -> lower=-0.785375 upper=0.785375 effort=0.0 velocity=0.0
- joint RightUpperArm_RightLowerArm: limit lower=-0.31415000000000004 upper=0.0 effort=0.0 velocity=0.0 -> lower=-0.5235833333333334 upper=0.0 effort=0.0 velocity=0.0
