Commit message: sim

File: body.urdf (robot description, URDF)
Before this commit: robot robot, 7 links, 6 joints
Links:
- removed link Torso
- added link Hips, mass 2.5; collision box size=0.8 1.0 0.5; visual box size=0.8 1.0 0.5
- added link LowerTorso, mass 1.25; collision box size=0.675 0.875 0.25; visual box size=0.675 0.875 0.25
- added link MidTorso, mass 1; collision box size=0.55 0.75 0.25; visual box size=0.55 0.75 0.25
- added link UpperTorso, mass 1; collision box size=0.65 0.85 0.5; visual box size=0.65 0.85 0.5
- link LeftFoot: mass 1 -> 1.25; geometry collision box size=0.675 0.675 0.225; visual box size=0.675 0.675 0.225
- link LeftLeg: mass 1 -> 3; geometry collision box size=0.45 0.45 2.25; visual box size=0.45 0.45 2.25
- link LeftLowerLeg: mass 1 -> 1.5; geometry collision box size=0.35 0.35 1.625; visual box size=0.35 0.35 1.625
- link RightFoot: mass 1 -> 1.25; geometry collision box size=0.675 0.675 0.225; visual box size=0.675 0.675 0.225
- link RightLeg: mass 1 -> 3; geometry collision box size=0.45 0.45 2.25; visual box size=0.45 0.45 2.25
- link RightLowerLeg: mass 1 -> 1.5; geometry collision box size=0.35 0.35 1.625; visual box size=0.35 0.35 1.625
Joints:
- removed joint Torso_LeftLeg
- removed joint Torso_RightLeg
- added joint Hips_LeftLeg: type revolute, parent Hips, child LeftLeg, origin xyz=0.0 0.5 4.0 rpy=0 0 0, axis 0 1 0, limit lower=-1.57075 upper=1.57075 effort=0.0 velocity=0.0
- added joint Hips_LowerTorso: type revolute, parent Hips, child LowerTorso, origin xyz=0.0 0.0 4.25 rpy=0 0 0, axis 0 1 0, limit lower=-0.2617916666666667 upper=0.2617916666666667 effort=0.0 velocity=0.0
- added joint Hips_RightLeg: type revolute, parent Hips, child RightLeg, origin xyz=0.0 -0.5 4.0 rpy=0 0 0, axis 0 1 0, limit lower=-1.57075 upper=1.57075 effort=0.0 velocity=0.0
- added joint LowerTorso_MidTorso: type revolute, parent LowerTorso, child MidTorso, origin xyz=0.0 0.0 0.25 rpy=0 0 0, axis 0 1 0, limit lower=0.0 upper=0.0 effort=0.0 velocity=0.0
- added joint MidTorso_UpperTorso: type revolute, parent MidTorso, child UpperTorso, origin xyz=0.0 0.0 0.25 rpy=0 0 0, axis 0 1 0, limit lower=-0.2617916666666667 upper=0.2617916666666667 effort=0.0 velocity=0.0
- joint LeftLeg_LeftLowerLeg: limit lower=0.0 upper=0.785375 effort=0.0 velocity=0.0 -> lower=0.0 upper=3.1415 effort=0.0 velocity=0.0
- joint LeftLowerLeg_LeftFoot: limit lower=-0.785375 upper=1.57075 effort=0.0 velocity=0.0 -> lower=-0.5235833333333334 upper=0.31415000000000004 effort=0.0 velocity=0.0
- joint RightLeg_RightLowerLeg: limit lower=0.0 upper=0.785375 effort=0.0 velocity=0.0 -> lower=0.0 upper=3.1415 effort=0.0 velocity=0.0
- joint RightLowerLeg_RightFoot: limit lower=-0.785375 upper=1.57075 effort=0.0 velocity=0.0 -> lower=-0.5235833333333334 upper=0.31415000000000004 effort=0.0 velocity=0.0

Commit message: silliness

File: body.urdf (robot description, URDF)
Before this commit: robot robot, 16 links, 15 joints
Links:
- link LeftFoot: mass 1 -> 1.5
- link LeftLeg: mass 2.75 -> 3.5
- link LeftLowerLeg: mass 1.5 -> 2.75
- link LeftUpperArm: mass 1.5 -> 2.0
- link RightFoot: mass 1 -> 1.5
- link RightLeg: mass 2.75 -> 3.5
- link RightLowerLeg: mass 1.5 -> 2.75
- link RightUpperArm: mass 1.5 -> 2.0
Joints:
- joint Hips_LeftLeg: limit lower=-1.57075 upper=1.57075 effort=0.0 velocity=0.0 -> lower=0.785375 upper=-0.785375 effort=0.0 velocity=0.0
- joint Hips_RightLeg: limit lower=-1.57075 upper=1.57075 effort=0.0 velocity=0.0 -> lower=-0.785375 upper=0.785375 effort=0.0 velocity=0.0
- joint LeftUpperArm_LeftLowerArm: limit lower=-0.5235833333333334 upper=0.0 effort=0.0 velocity=0.0 -> lower=0.5235833333333334 upper=0.0 effort=0.0 velocity=0.0
- joint RightUpperArm_RightLowerArm: limit lower=-0.5235833333333334 upper=0.0 effort=0.0 velocity=0.0 -> lower=0.5235833333333334 upper=0.0 effort=0.0 velocity=0.0

Commit message: lots of stuff

File: body.urdf (robot description, URDF)
Before this commit: robot robot, 16 links, 15 joints
Links:
- link LeftLowerArm: geometry collision box size=0.3 0.3 0.95; visual box size=0.3 0.3 0.95
- link LeftShoulder: geometry collision box size=0.55 1.125 0.25; visual box size=0.55 1.125 0.25
- link LeftUpperArm: geometry collision box size=0.35 0.35 1.0; visual box size=0.35 0.35 1.0
- link LowerTorso: mass 1.25 -> 1.0
- link RightLowerArm: geometry collision box size=0.3 0.3 0.95; visual box size=0.3 0.3 0.95
- link RightShoulder: geometry collision box size=0.55 1.125 0.25; visual box size=0.55 1.125 0.25
- link RightUpperArm: geometry collision box size=0.35 0.35 1.0; visual box size=0.35 0.35 1.0
Joints:
- joint Hips_LeftLeg: limit lower=0.785375 upper=-0.785375 effort=0.0 velocity=0.0 -> lower=-1.5707963267948966 upper=0.7853981633974483 effort=0.0 velocity=0.0
- joint Hips_LowerTorso: limit lower=-0.2617916666666667 upper=0.2617916666666667 effort=0.0 velocity=0.0 -> lower=-0.2617993877991494 upper=0.2617993877991494 effort=0.0 velocity=0.0; type revolute -> fixed
- joint Hips_RightLeg: limit lower=-0.785375 upper=0.785375 effort=0.0 velocity=0.0 -> lower=-1.5707963267948966 upper=0.7853981633974483 effort=0.0 velocity=0.0
- joint LeftLeg_LeftLowerLeg: limit lower=0.0 upper=3.1415 effort=0.0 velocity=0.0 -> lower=0.0 upper=1.5707963267948966 effort=0.0 velocity=0.0
- joint LeftLowerLeg_LeftFoot: limit lower=-0.785375 upper=0.3926875 effort=0.0 velocity=0.0 -> lower=-0.5235987755982988 upper=0.2617993877991494 effort=0.0 velocity=0.0
- joint LeftShoulder_LeftUpperArm: limit lower=0.785375 upper=-0.785375 effort=0.0 velocity=0.0 -> lower=-0.39269908169872414 upper=0.39269908169872414 effort=0.0 velocity=0.0
- joint LeftUpperArm_LeftLowerArm: limit lower=0.5235833333333334 upper=0.0 effort=0.0 velocity=0.0 -> lower=-0.5235987755982988 upper=0.0 effort=0.0 velocity=0.0
- joint LowerTorso_MidTorso: type revolute -> fixed
- joint MidTorso_UpperTorso: limit lower=-0.2617916666666667 upper=0.2617916666666667 effort=0.0 velocity=0.0 -> lower=-0.2617993877991494 upper=0.2617993877991494 effort=0.0 velocity=0.0
- joint RightLeg_RightLowerLeg: limit lower=0.0 upper=3.1415 effort=0.0 velocity=0.0 -> lower=0.0 upper=1.5707963267948966 effort=0.0 velocity=0.0
- joint RightLowerLeg_RightFoot: limit lower=-0.785375 upper=0.3926875 effort=0.0 velocity=0.0 -> lower=-0.5235987755982988 upper=0.2617993877991494 effort=0.0 velocity=0.0
- joint RightShoulder_RightUpperArm: limit lower=-0.785375 upper=0.785375 effort=0.0 velocity=0.0 -> lower=-0.39269908169872414 upper=0.39269908169872414 effort=0.0 velocity=0.0
- joint RightUpperArm_RightLowerArm: limit lower=0.5235833333333334 upper=0.0 effort=0.0 velocity=0.0 -> lower=-0.5235987755982988 upper=0.0 effort=0.0 velocity=0.0

Commit message: debugging

File: body.urdf (robot description, URDF)
Before this commit: robot robot, 16 links, 15 joints
Links:
- removed link LeftLowerArm
- removed link LeftShoulder
- removed link LeftUpperArm
- removed link RightLowerArm
- removed link RightShoulder
- removed link RightUpperArm
- removed link UpperTorso
Joints:
- removed joint LeftShoulder_LeftUpperArm
- removed joint LeftUpperArm_LeftLowerArm
- removed joint MidTorso_UpperTorso
- removed joint RightShoulder_RightUpperArm
- removed joint RightUpperArm_RightLowerArm
- removed joint UpperTorso_LeftShoulder
- removed joint UpperTorso_RightShoulder

Commit message: more gens

File: body.urdf (robot description, URDF)
Before this commit: robot robot, 16 links, 15 joints
Links:
- removed link LowerTorso
- removed link MidTorso
- removed link UpperTorso
- added link Torso, mass 1.0; collision box size=0.55 0.65 1.0; visual box size=0.55 0.65 1.0
- link LeftShoulder: geometry collision box size=0.55 1.0 0.25; visual box size=0.55 1.0 0.25
- link RightShoulder: geometry collision box size=0.55 1.0 0.25; visual box size=0.55 1.0 0.25
Joints:
- removed joint Hips_LowerTorso
- removed joint LowerTorso_MidTorso
- removed joint MidTorso_UpperTorso
- removed joint UpperTorso_LeftShoulder
- removed joint UpperTorso_RightShoulder
- added joint Hips_Torso: type fixed, parent Hips, child Torso, origin xyz=0.0 0.0 4.25 rpy=0 0 0, axis 0 1 0, limit lower=-0.2617993877991494 upper=0.2617993877991494 effort=0.0 velocity=0.0
- added joint Torso_LeftShoulder: type revolute, parent Torso, child LeftShoulder, origin xyz=0.0 0.0 0.625 rpy=0 0 0, axis 0 0 1, limit lower=0.0 upper=0.0 effort=0.0 velocity=0.0
- added joint Torso_RightShoulder: type revolute, parent Torso, child RightShoulder, origin xyz=0.0 0.0 0.625 rpy=0 0 0, axis 0 0 1, limit lower=0.0 upper=0.0 effort=0.0 velocity=0.0
- joint Hips_LeftLeg: limit lower=-1.5707963267948966 upper=0.7853981633974483 effort=0.0 velocity=0.0 -> lower=-1.5707963267948966 upper=1.5707963267948966 effort=0.0 velocity=0.0
- joint Hips_RightLeg: limit lower=-1.5707963267948966 upper=0.7853981633974483 effort=0.0 velocity=0.0 -> lower=-1.5707963267948966 upper=1.5707963267948966 effort=0.0 velocity=0.0

Commit message: simple body

File: body.urdf (robot description, URDF)
Before this commit: robot robot, 14 links, 13 joints
Links:
- removed link LeftShoulder
- removed link RightShoulder
- added link Shoulders, mass 1; collision box size=0.55 2.0 0.25; visual box size=0.55 2.0 0.25
Joints:
- removed joint LeftShoulder_LeftUpperArm
- removed joint RightShoulder_RightUpperArm
- removed joint Torso_LeftShoulder
- removed joint Torso_RightShoulder
- added joint Shoulders_LeftUpperArm: type revolute, parent Shoulders, child LeftUpperArm, origin xyz=0.0 -1.0 0.125 rpy=0 0 0, axis 1 1 0, limit lower=-0.39269908169872414 upper=0.39269908169872414 effort=0.0 velocity=0.0
- added joint Shoulders_RightUpperArm: type revolute, parent Shoulders, child RightUpperArm, origin xyz=0.0 1.0 0.125 rpy=0 0 0, axis 1 1 0, limit lower=-0.39269908169872414 upper=0.39269908169872414 effort=0.0 velocity=0.0
- added joint Torso_Shoulders: type revolute, parent Torso, child Shoulders, origin xyz=0.0 0.0 1.0 rpy=0 0 0, axis 0 0 1, limit lower=0.0 upper=0.0 effort=0.0 velocity=0.0
- joint Hips_LeftLeg: limit lower=-1.5707963267948966 upper=1.5707963267948966 effort=0.0 velocity=0.0 -> lower=-1.5707963267948966 upper=0.7853981633974483 effort=0.0 velocity=0.0
- joint Hips_RightLeg: limit lower=-1.5707963267948966 upper=1.5707963267948966 effort=0.0 velocity=0.0 -> lower=-1.5707963267948966 upper=0.7853981633974483 effort=0.0 velocity=0.0
- joint LeftLeg_LeftLowerLeg: limit lower=0.0 upper=1.5707963267948966 effort=0.0 velocity=0.0 -> lower=0.0 upper=0.5235987755982988 effort=0.0 velocity=0.0
- joint RightLeg_RightLowerLeg: limit lower=0.0 upper=1.5707963267948966 effort=0.0 velocity=0.0 -> lower=0.0 upper=0.5235987755982988 effort=0.0 velocity=0.0

Commit message: adjust body

File: body.urdf (robot description, URDF)
Before this commit: robot robot, 13 links, 12 joints
Links:
- link Shoulders: geometry collision box size=0.5 2.0 0.25; visual box size=0.5 2.0 0.25
Joints:
- joint Shoulders_LeftUpperArm: origin xyz=0.0 -1.0 0.125 rpy=0 0 0 -> xyz=0.0 -0.95 0.125 rpy=0 0 0
- joint Shoulders_RightUpperArm: origin xyz=0.0 1.0 0.125 rpy=0 0 0 -> xyz=0.0 0.95 0.125 rpy=0 0 0

Commit message: sin value to sensor

File: body.urdf (robot description, URDF)
Before this commit: robot robot, 13 links, 12 joints
Joints:
- joint LeftUpperArm_LeftLowerArm: limit lower=-0.5235987755982988 upper=0.0 effort=0.0 velocity=0.0 -> lower=-0.7853981633974483 upper=0.0 effort=0.0 velocity=0.0
- joint RightUpperArm_RightLowerArm: limit lower=-0.5235987755982988 upper=0.0 effort=0.0 velocity=0.0 -> lower=-0.7853981633974483 upper=0.0 effort=0.0 velocity=0.0
- joint Shoulders_LeftUpperArm: limit lower=-0.39269908169872414 upper=0.39269908169872414 effort=0.0 velocity=0.0 -> lower=-0.7853981633974483 upper=0.7853981633974483 effort=0.0 velocity=0.0
- joint Shoulders_RightUpperArm: limit lower=-0.39269908169872414 upper=0.39269908169872414 effort=0.0 velocity=0.0 -> lower=-0.7853981633974483 upper=0.7853981633974483 effort=0.0 velocity=0.0

Commit message: edits

File: body.urdf (robot description, URDF)
Before this commit: robot robot, 9 links, 8 joints
Joints:
- joint Hips_LeftLeg: limit lower=-1.5707963267948966 upper=0.7853981633974483 effort=0.0 velocity=0.0 -> lower=-0.7853981633974483 upper=0.5235987755982988 effort=0.0 velocity=0.0
- joint Hips_RightLeg: limit lower=-1.5707963267948966 upper=0.7853981633974483 effort=0.0 velocity=0.0 -> lower=-0.7853981633974483 upper=0.5235987755982988 effort=0.0 velocity=0.0
- joint LeftLeg_LeftLowerLeg: limit lower=0.0 upper=1.5707963267948966 effort=0.0 velocity=0.0 -> lower=0.0 upper=0.5235987755982988 effort=0.0 velocity=0.0
- joint RightLeg_RightLowerLeg: limit lower=0.0 upper=1.5707963267948966 effort=0.0 velocity=0.0 -> lower=0.0 upper=0.5235987755982988 effort=0.0 velocity=0.0

Commit message: adjust

File: body.urdf (robot description, URDF)
Before this commit: robot robot, 13 links, 12 joints
Joints:
- joint Hips_LeftLeg: limit lower=-1.5707963267948966 upper=0.7853981633974483 effort=0.0 velocity=0.0 -> lower=-0.5235987755982988 upper=0.5235987755982988 effort=0.0 velocity=0.0
- joint Hips_RightLeg: limit lower=-1.5707963267948966 upper=0.7853981633974483 effort=0.0 velocity=0.0 -> lower=-0.5235987755982988 upper=0.5235987755982988 effort=0.0 velocity=0.0

Commit message: img

File: body.urdf (robot description, URDF)
Before this commit: robot robot, 9 links, 8 joints
Joints:
- joint Hips_LeftLeg: limit lower=-0.7853981633974483 upper=0.5235987755982988 effort=0.0 velocity=0.0 -> lower=-0.5235987755982988 upper=0.5235987755982988 effort=0.0 velocity=0.0
- joint Hips_RightLeg: limit lower=-0.7853981633974483 upper=0.5235987755982988 effort=0.0 velocity=0.0 -> lower=-0.5235987755982988 upper=0.5235987755982988 effort=0.0 velocity=0.0
